File: SCK.brd (EAGLE design)
At the start: 42 x 35 mm, 46 parts

Commit message: Added 3D Models
Parts:
- removed RTC1: DS3231M, SparkFun-Clocks:SO08
- removed U$1: ATTINY84, SparkFun-IC-Microcontroller:SO14
- added U$3: DS3231M, SCK_custom:SOIC127P600X175-8
- added U$4: MAX7219, SCK_custom:SOIC127P1032X265-24
- U$2: value MAX7219 -> ATTINY84; device CLK_IC:SOIC24L -> SCK_custom:SOIC127P599X175-14
- moved U$2 21.2 mm to (32.0, 14.5), turned to 0 degrees
- moved C4 0.50 mm to (32.0, 32.0)
Connections:
- net GND: now also U$2.14, U$3.2, U$3.5, U$4.4, U$4.9; no longer RTC1.2, RTC1.5, U$1.14, U$2.4, U$2.9
- net GRID1: now also U$4.2; no longer U$2.2
- net GRID2: now also U$4.11; no longer U$2.11
- net GRID3: now also U$4.6; no longer U$2.6
- net GRID4: now also U$4.7; no longer U$2.7
- net N$2: now also U$4.18; no longer U$2.18
- net PA0: now also U$2.13; no longer U$1.13
- net PA1: now also U$2.12; no longer U$1.12
- net PA2: now also U$2.11, U$4.12; no longer U$1.11, U$2.12
- net PA3: now also U$2.10, U$4.13; no longer U$1.10, U$2.13
- net PA4: now also U$2.9, U$3.8; no longer RTC1.8, U$1.9
- net PA5: now also U$2.8, U$4.1; no longer U$1.8, U$2.1
- net PA6: now also U$2.7, U$3.7; no longer RTC1.7, U$1.7
- net PA7: now also U$2.6; no longer U$1.6
- net PB0: now also U$2.2; no longer U$1.2
- net PB1: now also U$2.3; no longer U$1.3
- net PB2: now also U$2.5; no longer U$1.5
- net PB3: now also U$2.4; no longer U$1.4
- net SEG1: now also U$4.14; no longer U$2.14
- net SEG2: now also U$4.16; no longer U$2.16
- net SEG3: now also U$4.20; no longer U$2.20
- net SEG4: now also U$4.23; no longer U$2.23
- net SEG5: now also U$4.21; no longer U$2.21
- net SEG6: now also U$4.15; no longer U$2.15
- net SEG7: now also U$4.17; no longer U$2.17
- net SEG8: now also U$4.22; no longer U$2.22
- net VCC: now also U$2.1, U$3.6, U$4.19; no longer RTC1.6, U$1.1, U$2.19
Routing:
- net PB3: track 7.06 -> 0.00 mm, vias 1 -> 0
- net VCC: track 129.0 -> 130.8 mm
- net GRID3: track 36.6 -> 35.6 mm
- net PA3: track 60.9 -> 61.8 mm
- net PA4: track 26.6 -> 27.4 mm
- net SEG4: track 41.9 -> 42.6 mm
- net SEG7: track 39.1 -> 39.8 mm
- net SEG2: track 35.8 -> 36.5 mm
- net N$2: track 16.7 -> 17.3 mm
- net SEG8: track 45.2 -> 45.9 mm
- net GRID4: track 36.2 -> 35.6 mm
- net GND: track 16.0 -> 15.9 mm, vias 20 -> 19
