File: SCK.sch (EAGLE design)
At the start: 46 parts

Commit message: Added 3D Models
Parts:
- removed RTC1: DS3231M, SparkFun-Clocks:DS3231M
- removed U$1: ATTINY84, SparkFun-IC-Microcontroller:ATTINY84
- added U$3: DS3231M, SCK_custom:DS3231M
- added U$4: MAX7219, SCK_custom:MAX7219
- U$2: value MAX7219 -> ATTINY84; device CLK_IC:MAX7219 -> SCK_custom:ATTINY84
Connections:
- net GND: now also U$3.GND, U$3.VCC, U$4.GND; no longer RTC1.GND, RTC1.VCC, U$1.GND
- net GRID1: now also U$4.DIG0; no longer U$2.DIG0
- net GRID2: now also U$4.DIG1; no longer U$2.DIG1
- net GRID3: now also U$4.DIG2; no longer U$2.DIG2
- net GRID4: now also U$4.DIG3; no longer U$2.DIG3
- net N$2: now also U$4.ISET; no longer U$2.ISET
- net PA0: now also U$2.(PCINT0/AREF/ADC0)PA0; no longer U$1.(PCINT0/AREF/ADC0)PA0
- net PA1: now also U$2.(PCINT1/AIN0/ADC1)PA1; no longer U$1.(PCINT1/AIN0/ADC1)PA1
- net PA2: now also U$2.(PCINT2/AIN1/ADC2)PA2, U$4.CS; no longer U$1.(PCINT2/AIN1/ADC2)PA2, U$2.CS
- net PA3: now also U$2.(PCINT3/T0/ADC3)PA3, U$4.CLK; no longer U$1.(PCINT3/T0/ADC3)PA3, U$2.CLK
- net PA4: now also U$2.(PCINT4/T1/SCL/USCK/ADC4)PA4, U$3.SCL; no longer RTC1.SCL, U$1.(PCINT4/T1/SCL/USCK/ADC4)PA4
- net PA5: now also U$2.(PCINT5/OC1B/MISO/DO/ADC5)PA5, U$4.DIN; no longer U$1.(PCINT5/OC1B/MISO/DO/ADC5)PA5, U$2.DIN
- net PA6: now also U$2.(PCINT6/OC1A/SDA/MOSI/ADC6)PA6, U$3.SDA; no longer RTC1.SDA, U$1.(PCINT6/OC1A/SDA/MOSI/ADC6)PA6
- net PA7: now also U$2.(PCINT7/ICP/OC0B/ADC7)PA7; no longer U$1.(PCINT7/ICP/OC0B/ADC7)PA7
- net PB0: now also U$2.(PCINT8/XTAL1/CLKI)PB0; no longer U$1.(PCINT8/XTAL1/CLKI)PB0
- net PB1: now also U$2.(PCINT9/XTAL2)PB1; no longer U$1.(PCINT9/XTAL2)PB1
- net PB2: now also U$2.(PCINT10/INT0/OC0A/CKOUT)PB2; no longer U$1.(PCINT10/INT0/OC0A/CKOUT)PB2
- net PB3: now also U$2.(PCINT11/~RESET/DW)PB3; no longer U$1.(PCINT11/~RESET/DW)PB3
- net SEG1: now also U$4.SEGA; no longer U$2.SEGA
- net SEG2: now also U$4.SEGB; no longer U$2.SEGB
- net SEG3: now also U$4.SEGC; no longer U$2.SEGC
- net SEG4: now also U$4.SEGD; no longer U$2.SEGD
- net SEG5: now also U$4.SEGE; no longer U$2.SEGE
- net SEG6: now also U$4.SEGF; no longer U$2.SEGF
- net SEG7: now also U$4.SEGG; no longer U$2.SEGG
- net SEG8: now also U$4.SEGDP; no longer U$2.SEGDP
- net VCC: now also U$3.VBAT, U$4.VCC; no longer RTC1.VBAT, U$1.VCC
Other:
- moved on the sheet: C4
